File: Eagle Design/V1 REV1/cartridge_reader.brd (EAGLE design)
At the start: 68.6 x 30.5 mm, 21 parts, among them IC1 AT90USB1287-AU

Commit message: lufa and cartridge dumper
Parts:
- added R4: 10kOhm, rcl:R0603
- added S2: (no value), SparkFun-Electromechanical:SWITCH-SPST-SMD-A
- R3: value 1kOhm -> 100Ohm
- moved S1 4.49 mm to (57.7, 16.5), turned to 90 degrees
Connections:
- new net N$43: R3.1, S2.3
- net N$26: now also R4.1, S2.1, S2.2; no longer R3.1
- net VCC: now also R4.2
Routing:
- net N$26: track 14.7 -> 13.6 mm
Changed lines of the file:
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@@
 <attribute name="VALUE" x="5.08" y="17.907" size="0.8128" layer="25"/>
 </element>
-<element name="R3" library="rcl" package="R0603" value="1kOhm" x="45.9486" y="21.5392" smashed="yes">
+<element name="R3" library="rcl" package="R0603" value="100Ohm" x="45.9486" y="21.5392" smashed="yes">
 <attribute name="NAME" x="47.8536" y="21.1582" size="0.8128" layer="25"/>
 <attribute name="VALUE" x="44.7421" y="22.3802" size="0.8128" layer="25"/>
@@
 <attribute name="NAME" x="6.5931" y="19.492" size="0.8128" layer="25"/>
 </element>
-<element name="S1" library="SparkFun-Electromechanical" package="TACTILE-SWITCH-1101NE" value="SWITCH-MOMENTARY-2-SMD-1101NE" x="60.96" y="19.558" smashed="yes" rot="R180"/>
+<element name="S1" library="SparkFun-Electromechanical" package="TACTILE-SWITCH-1101NE" value="SWITCH-MOMENTARY-2-SMD-1101NE" x="57.658" y="16.51" smashed="yes" rot="R90"/>
 <element name="JP4" library="adafruit" package="1X01" value="" x="62.23" y="28.956" smashed="yes">
 <attribute name="VALUE" x="60.96" y="25.781" size="1.27" layer="27"/>
@@
 <attribute name="VALUE" x="16.002" y="10.414" size="1.27" layer="27" ratio="10" rot="R180"/>
 </element>
+<element name="S2" library="SparkFun-Electromechanical" package="SWITCH-SPST-SMD-A" value="" x="66.675" y="21.59" rot="R270"/>
+<element name="R4" library="rcl" package="R0603" value="10kOhm" x="62.23" y="24.13" rot="R180"/>
 </elements>
 <signals>
@@
 <wire x1="59.194" y1="2.933" x2="57.54" y2="2.933" width="0.4064" layer="1"/>
 <wire x1="59.96" y1="5.08" x2="59.96" y2="3.699" width="0.4064" layer="1"/>
+<contactref element="R4" pad="2"/>
+<wire x1="61.38" y1="24.13" x2="12.446" y2="7.239" width="0" layer="19" extent="1-1"/>
 </signal>
 <signal name="N$1">
@@
 <via x="57.785" y="21.311" extent="1-16" drill="0.3302"/>
 <wire x1="57.785" y1="21.311" x2="57.785" y2="19.964" width="0.1524" layer="1"/>
-<wire x1="57.81" y1="19.558" x2="57.785" y2="19.964" width="0.1524" layer="1"/>
+<wire x1="57.658" y1="19.66" x2="57.785" y2="19.964" width="0.1524" layer="1"/>
 </signal>
 <signal name="N$30">
@@
 <signal name="N$26">
 <contactref element="IC1" pad="43"/>
-<contactref element="R3" pad="1"/>
 <wire x1="30.70899375" y1="22.357725" x2="44.280075" y2="22.357725" width="0.1524" layer="1"/>
-<wire x1="44.280075" y1="22.357725" x2="45.0986" y2="21.5392" width="0.1524" layer="1"/>
+<contactref element="S2" pad="2"/>
+<contactref element="R4" pad="1"/>
+<contactref element="S2" pad="1"/>
+<wire x1="64.925" y1="22.34" x2="64.925" y2="23.84" width="0" layer="19" extent="1-1"/>
+<wire x1="63.08" y1="24.13" x2="64.925" y2="23.84" width="0" layer="19" extent="1-1"/>
+<wire x1="44.280075" y1="22.357725" x2="63.08" y2="24.13" width="0" layer="19" extent="1-1"/>
 </signal>
 <signal name="N$28">
@@
 <wire x1="10.985" y1="4.488" x2="11.04" y2="4.433" width="0.4064" layer="1"/>
 </signal>
+<signal name="N$43">
+<contactref element="S2" pad="3"/>
+<contactref element="R3" pad="1"/>
+<wire x1="45.0986" y1="21.5392" x2="64.925" y2="19.34" width="0" layer="19" extent="1-1"/>
+</signal>
 </signals>
